Commit message: Adding IKFast plugin and ...
Modified description (may not have been completely necessary)(needs review). 
Changed meshes. New offsets for openrave dae creation.
Created IKFast solver and MoveIt plugin.
TODO: Functional gripper controller.

File: widowx_arm/widowx_arm_description/urdf/widowx.urdf.xacro (robot description, xacro)
@@ -133,5 +133,5 @@
          </inertial>
       </link>
-      <link name="${prefix}gripper_rail_link">
+      <!--link name="${prefix}gripper_rail_link">
          <visual>
             <origin xyz="0 0 0" rpy="0 0 1.57" />
@@ -152,8 +152,8 @@
             <inertia ixx="1.0" ixy="0.0" ixz="0.0" iyy="1.0" iyz="0.0" izz="1.0" />
          </inertial>
-      </link>
-      <link name="${prefix}gripper_aux_link">
-      </link>
-      <link name="${prefix}gripper_1_link">
+      </link-->
+      <!--link name="${prefix}gripper_aux_link">
+      </link-->
+      <!--link name="${prefix}gripper_1_link">
          <visual>
             <origin xyz="0 -0.0007 0" rpy="0 0 1.57" />
@@ -194,5 +194,5 @@
             <inertia ixx="1.0" ixy="0.0" ixz="0.0" iyy="1.0" iyz="0.0" izz="1.0" />
          </inertial>
-      </link>
+      </link-->
       <!-- joints -->
       <joint name="${prefix}arm_base_joint" type="fixed">
@@ -237,5 +237,5 @@
          <limit lower="-2.617" upper="2.617" effort="0" velocity="1.571" />
       </joint>
-      <joint name="${prefix}joint_6" type="fixed">
+      <!--joint name="${prefix}joint_6" type="fixed">
          <origin xyz = "0 0 ${M_SCALE*43}" rpy="0 0 0" />
          <parent link="${prefix}wrist_2_link" />
@@ -243,13 +243,13 @@
          <axis xyz="0 0 1" />
          <limit lower="-0.31" upper="0.1" effort="0" velocity="0.5" />
-      </joint>
-      <joint name="${prefix}gripper_revolute_joint" type="revolute">
-         <origin xyz = "0 0 0" rpy="0 0 0" />
-         <parent link="${prefix}gripper_rail_link" />
+      </joint-->
+      <!--joint name="${prefix}gripper_revolute_joint" type="revolute">
+         <origin xyz = "0 0 0.065" rpy="0 0 0" />
+         <parent link="${prefix}wrist_2_link" />
          <child link="${prefix}gripper_aux_link" />
          <axis xyz="0 0 1" />
          <limit lower="-2.6" upper="2.6" effort="0" velocity="0.5" />
-      </joint>
-      <joint name="${prefix}gripper_prismatic_joint_1" type="prismatic">
+      </joint-->
+      <!--joint name="${prefix}gripper_prismatic_joint_1" type="prismatic">
          <origin xyz="0 0 0" rpy="0 0 0" />
          <parent link="${prefix}gripper_rail_link" />
@@ -265,5 +265,7 @@
          <axis xyz="0 1 0" />
          <limit lower="0" upper="0.027" effort="0" velocity="0.5" />
-      </joint>
+      </joint-->
+      <!-- gripper -->
+  <xacro:include filename="$(find widowx_arm_description)/urdf/widowx_gripper.xacro"/>
    </xacro:macro>
   <transmission name="tran1">
