Commit message: Improving block manipulation and sorting

File: widowx_arm/widowx_arm_description/urdf/sensor_sr300.urdf.xacro (robot description, xacro)
@@ -9,5 +9,5 @@
   <xacro:property name="sr300_cam_offset_px" value="0.330" />
   <xacro:property name="sr300_cam_offset_py" value="0.0" />
-  <xacro:property name="sr300_cam_offset_pz" value="0.380" />
+  <xacro:property name="sr300_cam_offset_pz" value="0.385" />
   <xacro:property name="sr300_cam_rgb_px" value="0.012"/>
   <xacro:property name="sr300_cam_rgb_py" value="0.003"/>

Commit message: Block sorting tweaks

File: widowx_arm/widowx_arm_description/urdf/sensor_sr300.urdf.xacro (robot description, xacro)
@@ -9,5 +9,5 @@
   <xacro:property name="sr300_cam_offset_px" value="0.330" />
   <xacro:property name="sr300_cam_offset_py" value="0.0" />
-  <xacro:property name="sr300_cam_offset_pz" value="0.385" />
+  <xacro:property name="sr300_cam_offset_pz" value="0.380" />
   <xacro:property name="sr300_cam_rgb_px" value="0.012"/>
   <xacro:property name="sr300_cam_rgb_py" value="0.003"/>
