Commit message: Update MoveIt setup

File: widowx_arm/widowx_arm_description/robots/widowx_arm_ikfast.urdf (robot description, URDF)
Before this commit: robot widowx_arm, 7 links, 6 joints
Links:
- added link gripper_link
Joints:
- added joint gripper_link_joint: type revolute, parent wrist_2_link, child gripper_link, origin xyz=0 0 0.110 rpy=0 0 0, axis 1 0 0, limit lower=-3.14 upper=3.14 effort=6 velocity=1

File: widowx_arm/widowx_arm_description/urdf/widowx.urdf.xacro (robot description, xacro)
@@ -53,15 +53,14 @@
       <link name="${prefix}biceps_link">
          <visual>
-			      <origin xyz="${M_SCALE*48.25} 0 ${M_SCALE*140}" rpy="0 0 0" />
-            <!--origin xyz="0 0 0" rpy="0 0 0" /-->
-            <geometry>
-               <mesh filename="package://widowx_arm_description/meshes/biceps_link.stl" />
-            </geometry>
-            <xacro:material_black />
-         </visual>
-         <collision>
-            <origin xyz="0 0 0" rpy="0 0 0" />
-            <geometry>
-               <mesh filename="package://widowx_arm_description/meshes/biceps_link.stl" />
+            <origin xyz="0 0 0" rpy="0 0 0" />
+            <geometry>
+               <mesh filename="package://widowx_arm_description/meshes/biceps_link.new.stl" />
+            </geometry>
+            <xacro:material_black />
+         </visual>
+         <collision>
+            <origin xyz="0 0 0" rpy="0 0 0" />
+            <geometry>
+               <mesh filename="package://widowx_arm_description/meshes/biceps_link.new.stl" />
             </geometry>
          </collision>
@@ -74,8 +73,7 @@
       <link name="${prefix}forearm_link">
          <visual>
-			      <origin xyz="0 0 ${M_SCALE*142.03}" rpy="0 0 0" />
-			<!--origin xyz="0 0 0" rpy="0 0 0" /-->
-            <geometry>
-               <mesh filename="package://widowx_arm_description/meshes/forearm_link.stl"/>
+            <origin xyz="0 0 0" rpy="0 0 0" />
+            <geometry>
+               <mesh filename="package://widowx_arm_description/meshes/forearm_link.new.stl"/>
             </geometry>
            <xacro:material_black />
@@ -84,5 +82,5 @@
             <origin xyz="0 0 0" rpy="0 0 0" />
             <geometry>
-               <mesh filename="package://widowx_arm_description/meshes/forearm_link.stl"/>
+               <mesh filename="package://widowx_arm_description/meshes/forearm_link.new.stl"/>
             </geometry>
          </collision>
@@ -115,14 +113,14 @@
       <link name="${prefix}wrist_2_link">
          <visual>
-            <origin xyz="0 0 ${M_SCALE*43}" rpy="0 0 0" />
-            <geometry>
-               <mesh filename="package://widowx_arm_description/meshes/wrist_2_link.stl"/>
-            </geometry>
-            <xacro:material_black />
-         </visual>
-         <collision>
-            <origin xyz="0 0 0" rpy="0 0 0" />
-            <geometry>
-               <mesh filename="package://widowx_arm_description/meshes/wrist_2_link.stl"/>
+            <origin xyz="0 0 0" rpy="0 0 0" />
+            <geometry>
+               <mesh filename="package://widowx_arm_description/meshes/wrist_2_link.new.stl"/>
+            </geometry>
+            <xacro:material_black />
+         </visual>
+         <collision>
+            <origin xyz="0 0 0" rpy="0 0 0" />
+            <geometry>
+               <mesh filename="package://widowx_arm_description/meshes/wrist_2_link.new.stl"/>
             </geometry>
          </collision>
@@ -206,5 +204,5 @@
          <child link="${prefix}shoulder_link" />
          <axis xyz="0 0 1" />
-         <limit lower="-2.617" upper="2.617" effort="0" velocity="0.785" />
+         <limit lower="-2.617" upper="2.617" effort="6" velocity="0.785" />
       </joint>
       <joint name="${prefix}joint_2" type="revolute">
@@ -214,5 +212,5 @@
          <child link="${prefix}biceps_link" />
          <axis xyz="0 1 0" />
-         <limit lower="-1.571" upper="1.571" effort="0" velocity="1.571" />
+         <limit lower="-1.571" upper="1.571" effort="6" velocity="1.571" />
       </joint>
       <joint name="${prefix}joint_3" type="revolute">
@@ -221,5 +219,5 @@
          <child link="${prefix}forearm_link" />
          <axis xyz="0 1 0" />
-         <limit lower="-1.571" upper="1.571" effort="0" velocity="1.571" />
+         <limit lower="-1.571" upper="1.571" effort="6" velocity="1.571" />
       </joint>
       <joint name="${prefix}joint_4" type="revolute">
@@ -228,5 +226,5 @@
          <child link="${prefix}wrist_1_link" />
          <axis xyz="0 1 0" />
-         <limit lower="-1.745" upper="1.745" effort="0" velocity="1.571" />
+         <limit lower="-1.745" upper="1.745" effort="6" velocity="1.571" />
       </joint>
       <joint name="${prefix}joint_5" type="revolute">
@@ -235,5 +233,5 @@
          <child link="${prefix}wrist_2_link" />
          <axis xyz="0 0 1" />
-         <limit lower="-2.617" upper="2.617" effort="0" velocity="1.571" />
+         <limit lower="-2.617" upper="2.617" effort="6" velocity="1.571" />
       </joint>
       <!--joint name="${prefix}joint_6" type="fixed">
@@ -242,5 +240,5 @@
          <child link="${prefix}gripper_rail_link" />
          <axis xyz="0 0 1" />
-         <limit lower="-0.31" upper="0.1" effort="0" velocity="0.5" />
+         <limit lower="-0.31" upper="0.1" effort="6" velocity="0.5" />
       </joint-->
       <!--joint name="${prefix}gripper_revolute_joint" type="revolute">
@@ -249,5 +247,5 @@
          <child link="${prefix}gripper_aux_link" />
          <axis xyz="0 0 1" />
-         <limit lower="-2.6" upper="2.6" effort="0" velocity="0.5" />
+         <limit lower="-2.6" upper="2.6" effort="6" velocity="0.5" />
       </joint-->
       <!--joint name="${prefix}gripper_prismatic_joint_1" type="prismatic">
@@ -256,5 +254,5 @@
          <child link="${prefix}gripper_1_link" />
          <axis xyz="0 -1 0" />
-         <limit lower="0" upper="0.027" effort="0" velocity="0.5" />
+         <limit lower="0" upper="0.027" effort="6" velocity="0.5" />
       </joint>
       <joint name="${prefix}gripper_prismatic_joint_2" type="prismatic">
@@ -264,8 +262,16 @@
          <mimic joint="${prefix}gripper_prismatic_joint_1" />
          <axis xyz="0 1 0" />
-         <limit lower="0" upper="0.027" effort="0" velocity="0.5" />
+         <limit lower="0" upper="0.027" effort="6" velocity="0.5" />
       </joint-->
       <!-- gripper -->
   <xacro:include filename="$(find widowx_arm_description)/urdf/widowx_gripper.xacro"/>
+  <!--link name="gripper_link"/>
+    <joint name="gripper_link_joint" type="revolute">
+      <origin xyz="0 0 0.110" rpy="0 0 0"/>
+      <parent link="${prefix}wrist_1_link" />
+      <child link="gripper_link"/>
+      <limit effort="6" velocity="1" lower="-3.14" upper="3.14"/>
+      <axis xyz="1 0 0"/>
+    </joint-->
    </xacro:macro>
   <transmission name="tran1">

File: widowx_arm/widowx_arm_description/urdf/widowx_gripper.xacro (robot description, xacro)
@@ -10,5 +10,5 @@
          </visual>
          <collision>
-            <origin xyz="0 0 0" rpy="0 0 0" />
+            <origin xyz="0 0 0" rpy="0 0 1.57" />
             <geometry>
                <mesh filename="package://widowx_arm_description/meshes/gripper_rail_link.stl"/>
@@ -21,6 +21,6 @@
          </inertial>
       </link>
-      <link name="${prefix}gripper_aux_link">
-      </link>
+      <!--link name="${prefix}gripper_aux_link">
+      </link-->
     <link name="${prefix}gripper_1_link">
          <visual>
@@ -32,5 +32,5 @@
          </visual>
          <collision>
-            <origin xyz="0 0 0" rpy="0 0 0" />
+            <origin xyz="0 -0.0007 0" rpy="0 0 1.57" />
             <geometry>
                <mesh filename="package://widowx_arm_description/meshes/gripper_hand_fixed_link.stl"/>
@@ -52,5 +52,5 @@
          </visual>
          <collision>
-            <origin xyz="0 0 0" rpy="0 0 0" />
+            <origin xyz="0 0.0007 0" rpy="0 0 -1.57" />
             <geometry>
                <mesh filename="package://widowx_arm_description/meshes/gripper_hand_fixed_link.stl"/>
@@ -70,5 +70,5 @@
          <limit lower="-0.31" upper="0.1" effort="0" velocity="0.5" />
       </joint>
-      <joint name="${prefix}gripper_revolute_joint" type="revolute">
+      <!--joint name="${prefix}gripper_revolute_joint" type="revolute">
          <origin xyz = "0 0 0.065" rpy="0 0 0" />
          <parent link="${prefix}wrist_2_link" />
@@ -76,13 +76,13 @@
          <axis xyz="0 0 1" />
          <limit lower="-2.6" upper="2.6" effort="0" velocity="0.5" />
-      </joint>
-    <joint name="${prefix}gripper_prismatic_joint_1" type="prismatic">
+      </joint-->
+    <joint name="${prefix}gripper_joint" type="prismatic">
          <origin xyz="0 0 0" rpy="0 0 0" />
          <parent link="${prefix}gripper_rail_link" />
          <child link="${prefix}gripper_1_link" />
          <axis xyz="0 -1 0" />
-         <limit lower="0" upper="0.027" effort="0" velocity="0.5" />
+         <limit lower="0" upper="0.032" effort="0" velocity="0.5" />
       </joint>
-      <joint name="${prefix}gripper_prismatic_joint_2" type="prismatic">
+      <!--joint name="${prefix}gripper_prismatic_joint_2" type="prismatic">
          <origin xyz="0 0 0" rpy="0 0 0" />
          <parent link="${prefix}gripper_rail_link" />
@@ -91,4 +91,9 @@
          <axis xyz="0 1 0" />
          <limit lower="0" upper="0.027" effort="0" velocity="0.5" />
+      </joint-->
+      <joint name="${prefix}gripper_prismatic_joint_2" type="fixed">
+         <origin xyz="0 0 0" rpy="0 0 0" />
+         <parent link="${prefix}gripper_rail_link" />
+         <child link="${prefix}gripper_2_link" />
       </joint>
 </robot>

Commit message: Cleaning up description

File: widowx_arm/widowx_arm_description/robots/widowx_arm_ikfast.urdf (robot description, URDF)
Before this commit: robot widowx_arm, 8 links, 7 joints
Links:
- removed link gripper_link
Joints:
- removed joint gripper_link_joint

File: widowx_arm/widowx_arm_description/urdf/sensor_sr300.urdf.xacro (robot description, xacro)
@@ -7,13 +7,7 @@
   </xacro:property>
   <!-- Intel SR300 parameters -->
-  <xacro:property name="sr300_cam_offset_px" value="0.2" />
+  <xacro:property name="sr300_cam_offset_px" value="0.330" />
   <xacro:property name="sr300_cam_offset_py" value="0.0" />
-  <xacro:property name="sr300_cam_offset_pz" value="0.370" />
-  <!--
-  <xacro:property name="sr300_cam_rgb_px" value="0.005"/>
-  <xacro:property name="sr300_cam_rgb_py" value="0.018"/>
-  <xacro:property name="sr300_cam_rgb_pz" value="0.013"/>
-  <xacro:property name="sr300_cam_depth_offset" value="0.01"/>
-  -->
+  <xacro:property name="sr300_cam_offset_pz" value="0.380" />
   <xacro:property name="sr300_cam_rgb_px" value="0.012"/>
   <xacro:property name="sr300_cam_rgb_py" value="0.003"/>
@@ -26,5 +20,5 @@
     <!-- camera_sr300 body -->
     <joint name="camera_joint" type="fixed">
-      <origin xyz="${sr300_cam_offset_px} ${sr300_cam_offset_py} ${sr300_cam_offset_pz}" rpy="0 1.57 0"/>
+      <origin xyz="${sr300_cam_offset_px} ${sr300_cam_offset_py} ${sr300_cam_offset_pz}" rpy="0 1.16 3.14"/>
       <parent link="${parent}"/>
       <child link="camera_sr300" />
@@ -34,5 +28,5 @@
        <origin xyz="0 0 0" rpy="0 0 0"/>
         <geometry>
-         <mesh filename="package://turtlebot2i_description/meshes/sensors/sr300.stl" />
+         <mesh filename="package://widowx_arm_description/meshes/sensors/sr300.stl" />
         </geometry>
         <xacro:insert_block name="material_black"/>
@@ -41,5 +35,5 @@
         <origin xyz="0.0 0.0 0.0" rpy="0 0 0"/>
         <geometry>
-          <mesh filename="package://turtlebot2i_description/meshes/sensors/sr300.stl" scale="2.0 2.0 2.0" />
+          <mesh filename="package://widowx_arm_description/meshes/sensors/sr300.stl" scale="2.0 2.0 2.0" />
         </geometry>
       </collision>
@@ -88,5 +82,5 @@
     </joint>
     <link name="camera_depth_optical_frame"/>
-  	<!-- Simulation sensor -->
+    <!-- Simulation sensor -->
     <gazebo reference="camera_sr300">
       <sensor type="depth" name="camera_sr300">
